File: right/zzsplit-right.kicad_pcb (KiCad board)
At the start: 2 copper layers, 160.9 x 98.9 mm, 73 parts, among them J1 OLED, J2 MJ-4PP-9-Lily58-cache, J3 OLED, SW1 SW_PUSH-MX_W_LED, SW10 SW_PUSH-MX_W_LED, SW11 SW_PUSH-MX_W_LED, SW12 SW_PUSH-MX_W_LED, SW13 SW_PUSH-MX_W_LED, SW14 SW_PUSH-MX_W_LED, SW15 SW_PUSH-MX_W_LED, SW16 SW_PUSH-MX_W_LED, SW17 SW_PUSH-MX_W_LED, SW18 SW_PUSH-MX_W_LED, SW19 SW_PUSH-MX_W_LED, SW2 SW_PUSH-MX_W_LED, SW20 SW_PUSH-MX_W_LED, SW21 SW_PUSH-MX_W_LED, SW22 SW_PUSH-MX_W_LED, SW23 SW_PUSH-MX_W_LED, SW24 SW_PUSH-MX_W_LED, SW25 SW_PUSH-MX_W_LED, SW26 SW_PUSH-MX_W_LED, SW27 SW_PUSH-MX_W_LED, SW28 SW_PUSH-MX_W_LED, SW29 SW_PUSH-MX_W_LED, SW3 SW_PUSH-MX_W_LED, SW30 SW_PUSH-MX_W_LED, SW31 SW_SPDT, SW32 SW_Push, SW4 SW_PUSH-MX_W_LED, SW5 SW_PUSH-MX_W_LED, SW6 SW_PUSH-MX_W_LED, SW7 SW_PUSH-MX_W_LED, SW8 SW_PUSH-MX_W_LED, SW9 SW_PUSH-MX_W_LED, U1 ProMicro

Commit message: holes
Parts:
- added ?: , , F.Cu at (97.8, 137.5)
- added ?: , , F.Cu at (112.5, 51.7)
- added ?: , , F.Cu at (184.1, 136.8)
- added ?: , , F.Cu at (242.0, 67.0)
Changed lines of the file:
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@@
       (layerselection 0x00010fc_ffffffff)
       (disableapertmacros false)
-      (usegerberextensions false)
-      (usegerberattributes true)
-      (usegerberadvancedattributes true)
-      (creategerberjobfile true)
+      (usegerberextensions true)
+      (usegerberattributes false)
+      (usegerberadvancedattributes false)
+      (creategerberjobfile false)
       (svguseinch false)
       (svgprecision 6)
-      (excludeedgelayer true)
+      (excludeedgelayer false)
       (plotframeref false)
       (viasonmask false)
@@
       (plotvalue true)
       (plotinvisibletext false)
-      (sketchpadsonfab false)
-      (subtractmaskfromsilk false)
+      (sketchpadsonfab true)
+      (subtractmaskfromsilk true)
       (outputformat 1)
       (mirror false)
-      (drillshape 1)
+      (drillshape 0)
       (scaleselection 1)
-      (outputdirectory "")
+      (outputdirectory "zzsplit-right/")
     )
   )
@@
       (net 36 "VDD") (pinfunction "VDD") (pintype "power_in"))
   )
+  (footprint "" (layer "F.Cu")
+    (at 97.78 137.48)
+    (fp_text reference "" (at 0 0) (layer "F.SilkS")
+      (effects (font (size 1.27 1.27) (thickness 0.15)))
+    )
+    (fp_text value "" (at 0 0) (layer "F.SilkS")
+      (effects (font (size 1.27 1.27) (thickness 0.15)))
+    )
+    (pad "" thru_hole circle locked (at 0 0 90) (size 4.7 4.7) (drill 4.1) (layers *.Cu *.Mask "Dwgs.User")
+      (clearance 0.3))
+  )
   (footprint "SofleRGB:SK6812MINI_and_cherry" (layer "F.Cu")
     (at 218.05 96.24 180)
@@
     )
   )
+  (footprint "" (layer "F.Cu")
+    (at 112.46 51.67)
+    (fp_text reference "" (at 0 0) (layer "F.SilkS")
+      (effects (font (size 1.27 1.27) (thickness 0.15)))
+    )
+    (fp_text value "" (at 0 0) (layer "F.SilkS")
+      (effects (font (size 1.27 1.27) (thickness 0.15)))
+    )
+    (pad "" thru_hole circle locked (at 0 0 90) (size 4.7 4.7) (drill 4.1) (layers *.Cu *.Mask "Dwgs.User")
+      (clearance 0.3))
+  )
   (footprint "SofleRGB:SK6812MINI_and_cherry" (layer "F.Cu")
     (at 127.57 58.13 180)
@@
     )
   )
+  (footprint "" (layer "F.Cu")
+    (at 184.12 136.85)
+    (fp_text reference "" (at 0 0) (layer "F.SilkS")
+      (effects (font (size 1.27 1.27) (thickness 0.15)))
+    )
+    (fp_text value "" (at 0 0) (layer "F.SilkS")
+      (effects (font (size 1.27 1.27) (thickness 0.15)))
+    )
+    (pad "" thru_hole circle locked (at 0 0 90) (size 4.7 4.7) (drill 4.1) (layers *.Cu *.Mask "Dwgs.User")
+      (clearance 0.3))
+  )
   (footprint "SofleRGB:SK6812MINI_and_cherry" (layer "F.Cu")
     (at 203.77 58.14 180)
@@
     (fp_circle (center 9.6 0) (end 10.75 0) (layer "F.Fab") (width 0.1) (fill none))
     (fp_circle (center 0 0) (end 1.15 0) (layer "F.Fab") (width 0.1) (fill none))
-    (pad "1" thru_hole roundrect (at 0 0 180) (size 2.55 2.55) (drill 1.55) (layers *.Cu *.Mask) (roundrect_rratio 0.098039)
+    (pad "1" thru_hole roundrect (at 0 0 180) (size 2.55 2.55) (drill 1.55) (layers *.Cu *.Mask) (roundrect_rratio 0.09803882353)
       (net 86 "unconnected-(SW31-Pad1)") (pinfunction "A") (pintype "passive+no_connect"))
     (pad "2" thru_hole circle (at 4.8 0 180) (size 2.55 2.55) (drill 1.55) (layers *.Cu *.Mask)
@@
       (net 59 "Col4") (pintype "passive"))
   )
+  (footprint "" (layer "F.Cu")
+    (at 241.96 66.95)
+    (fp_text reference "" (at 0 0) (layer "F.SilkS")
+      (effects (font (size 1.27 1.27) (thickness 0.15)))
+    )
+    (fp_text value "" (at 0 0) (layer "F.SilkS")
+      (effects (font (size 1.27 1.27) (thickness 0.15)))
+    )
+    (pad "" thru_hole circle locked (at 0 0 90) (size 4.7 4.7) (drill 4.1) (layers *.Cu *.Mask "Dwgs.User")
+      (clearance 0.3))
+  )
   (footprint "logo:melogo" (layer "B.Cu")
     (at 239.73 56.97 180)
@@
   (via (at 180.68 71.85) (size 0.8) (drill 0.4) (layers "F.Cu" "B.Cu") (net 39))
   (via (at 137.93 50.56) (size 0.8) (drill 0.4) (layers "F.Cu" "B.Cu") (free) (net 39))
-  (via (at 112.22 53.36) (size 0.8) (drill 0.4) (layers "F.Cu" "B.Cu") (free) (net 39))
+  (via (at 116.94 50.14) (size 0.8) (drill 0.4) (layers "F.Cu" "B.Cu") (free) (net 39))
   (via (at 241.95 90.67) (size 0.8) (drill 0.4) (layers "F.Cu" "B.Cu") (net 39))
   (via (at 213.72 110.16) (size 0.8) (drill 0.4) (layers "F.Cu" "B.Cu") (net 39))
@@
     (polygon
       (pts
-        (xy 264.36 38.73)
-        (xy 264.5 153.49)
-        (xy 79.25 155.03)
-        (xy 84.72 36.76)
+        (xy 253.14 150.17)
+        (xy 80.49 151.35)
+        (xy 85.35 39.57)
+        (xy 252.55 39.57)
       )
     )
@@
     (polygon
       (pts
-        (xy 261.42 149.57)
-        (xy 84.3 151.53)
-        (xy 85 44.33)
-        (xy 259.46 43.21)
+        (xy 254.56 151.11)
+        (xy 80.02 152.18)
+        (xy 81.68 43)
+        (xy 253.73 41.22)
       )
     )
