File: left/zzsplit.kicad_pcb (KiCad board)
At the start: 2 copper layers, 160.9 x 98.9 mm, 73 parts, among them J1 OLED, J2 MJ-4PP-9-Lily58-cache, J3 Conn_01x02_Female, SW1 SW_PUSH-MX_W_LED, SW10 SW_PUSH-MX_W_LED, SW11 SW_PUSH-MX_W_LED, SW12 SW_PUSH-MX_W_LED, SW13 SW_PUSH-MX_W_LED, SW14 SW_PUSH-MX_W_LED, SW15 SW_PUSH-MX_W_LED, SW16 SW_PUSH-MX_W_LED, SW17 SW_PUSH-MX_W_LED, SW18 SW_PUSH-MX_W_LED, SW19 SW_PUSH-MX_W_LED, SW2 SW_PUSH-MX_W_LED, SW20 SW_PUSH-MX_W_LED, SW21 SW_PUSH-MX_W_LED, SW22 SW_PUSH-MX_W_LED, SW23 SW_PUSH-MX_W_LED, SW24 SW_PUSH-MX_W_LED, SW25 SW_PUSH-MX_W_LED, SW26 SW_PUSH-MX_W_LED, SW27 SW_PUSH-MX_W_LED, SW28 SW_PUSH-MX_W_LED, SW29 SW_PUSH-MX_W_LED, SW3 SW_PUSH-MX_W_LED, SW30 SW_PUSH-MX_W_LED, SW31 SW_SPDT, SW32 SW_Push, SW4 SW_PUSH-MX_W_LED, SW5 SW_PUSH-MX_W_LED, SW6 SW_PUSH-MX_W_LED, SW7 SW_PUSH-MX_W_LED, SW8 SW_PUSH-MX_W_LED, SW9 SW_PUSH-MX_W_LED, U1 ProMicro

Commit message: gerber files for right and left pcbs
Parts:
- renumbered ZzSplit to .V1
Other:
- board text added: "ZzSplit https://github.com/zzLinus/ZzSplit"
Changed lines of the file:
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@@
     (at 188.73 76.28 180)
     (attr board_only exclude_from_pos_files exclude_from_bom)
-    (fp_text reference "ZzSplit" (at -6.66 -11.75) (layer "B.SilkS")
-      (effects (font (size 3 3) (thickness 0.3)) (justify mirror))
+    (fp_text reference ".V1" (at 40.95 -64.11) (layer "B.SilkS")
+      (effects (font (size 1 1) (thickness 0.25)) (justify mirror))
     )
     (fp_text value "LOGO" (at 0.75 0) (layer "B.SilkS") hide
@@
   (gr_arc (start 214.11 43.490001) (mid 215.871312 44.225759) (end 216.600019 45.99) (layer "Edge.Cuts") (width 0.1))
   (gr_arc (start 55.7 45.96) (mid 56.432233 44.192233) (end 58.2 43.46) (layer "Edge.Cuts") (width 0.1))
+  (gr_text "ZzSplit      https://github.com/zzLinus/ZzSplit" (at 128.85 140.12) (layer "B.SilkS")
+    (effects (font (size 1.524 1.524) (thickness 0.3)) (justify mirror))
+  )
   (via (at 178.76 93.62) (size 0.8) (drill 0.4) (layers "F.Cu" "B.Cu") (free) (net 0))
   (segment (start 131.71 45.66) (end 132.47 46.42) (width 0.25) (layer "B.Cu") (net 1))

Commit message: holes
Parts:
- added ?: , , F.Cu at (187.9, 66.2)
- added ?: , , F.Cu at (83.7, 67.5)
- added ?: , , F.Cu at (183.3, 135.7)
- added ?: , , F.Cu at (64.9, 111.8)
Routing:
- net Row2: track 183.3 -> 181.6 mm
- net Row3: track 235.6 -> 235.0 mm
