File: left/zzsplit.kicad_sch (KiCad schematic)
At the start: 72 parts, among them J1 OLED, J2 MJ-4PP-9-Lily58-cache, J3 Conn_01x02_Female, SW1 SW_PUSH-MX_W_LED, SW10 SW_PUSH-MX_W_LED, SW11 SW_PUSH-MX_W_LED, SW12 SW_PUSH-MX_W_LED, SW13 SW_PUSH-MX_W_LED, SW14 SW_PUSH-MX_W_LED, SW15 SW_PUSH-MX_W_LED, SW16 SW_PUSH-MX_W_LED, SW17 SW_PUSH-MX_W_LED, SW18 SW_PUSH-MX_W_LED, SW19 SW_PUSH-MX_W_LED, SW2 SW_PUSH-MX_W_LED, SW20 SW_PUSH-MX_W_LED, SW21 SW_PUSH-MX_W_LED, SW22 SW_PUSH-MX_W_LED, SW23 SW_PUSH-MX_W_LED, SW24 SW_PUSH-MX_W_LED, SW25 SW_PUSH-MX_W_LED, SW26 SW_PUSH-MX_W_LED, SW27 SW_PUSH-MX_W_LED, SW28 SW_PUSH-MX_W_LED, SW29 SW_PUSH-MX_W_LED, SW3 SW_PUSH-MX_W_LED, SW30 SW_PUSH-MX_W_LED, SW31 SW_SPDT, SW32 SW_Push, SW4 SW_PUSH-MX_W_LED, SW5 SW_PUSH-MX_W_LED, SW6 SW_PUSH-MX_W_LED, SW7 SW_PUSH-MX_W_LED, SW8 SW_PUSH-MX_W_LED, SW9 SW_PUSH-MX_W_LED, U1 ProMicro

Commit message: fix rgb powerline problem and new 3 pin 2 channel switches
Parts:
- SW31: footprint Connector_Wire:SolderWire-0.75sqmm_1x03_P4.8mm_D1.25mm_OD2.3mm -> switch:switch-MSK-12C02-smd
Changed lines of the file:
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@@
     (property "Reference" "SW31" (id 0) (at 31.75 171.45 0))
     (property "Value" "SW_SPDT" (id 1) (at 31.75 173.99 0))
-    (property "Footprint" "Connector_Wire:SolderWire-0.75sqmm_1x03_P4.8mm_D1.25mm_OD2.3mm" (id 2) (at 31.75 179.07 0)
+    (property "Footprint" "switch:switch-MSK-12C02-smd" (id 2) (at 31.75 179.07 0)
       (effects (font (size 1.27 1.27)) hide)
     )
@@
     )
     (path "/474935d3-05af-4771-8ffc-37eaa5638224"
-      (reference "SW31") (unit 1) (value "SW_SPDT") (footprint "Connector_Wire:SolderWire-0.75sqmm_1x03_P4.8mm_D1.25mm_OD2.3mm")
+      (reference "SW31") (unit 1) (value "SW_SPDT") (footprint "switch:switch-MSK-12C02-smd")
     )
     (path "/d0bcdda7-579c-4020-b2d3-220f6e774609"
